File: hardware/NBIoT Wing.kicad_pcb (KiCad board)
At the start: 4 copper layers, 50.8 x 22.9 mm, 40 parts, among them J1 USB_B_Micro, J2 Conn_01x12_Female, J3 Conn_01x16_Female, J4 Conn_02x03_Odd_Even, J5 SIM_Card, Q1 BSS138, Q2 BSS138, Q3 BSS138, U1 FXMA108, U2 BC66

Commit message: kicad 8
Connections:
- net /~RESET renamed /~{RESET}
Other:
- net class Default removed
- net class PWR removed
